Commit message: tweak jackal lidar pose

File: arena_robots/components/lidar/jackal_default/lidar.urdf.xacro (robot description, xacro)
@@ -1,9 +1,7 @@
 <?xml version="1.0"?>
 <robot xmlns:xacro="http://www.ros.org/wiki/xacro">
-  <!-- Jackal's own bespoke gpu_lidar (link geometry, joint, gz sensor incl. its odd
-       internal <pose> duplicating the joint's own z-offset, an upstream
-       jackal_description quirk kept as-is). joint_name is separate from
-       frame because jackal's joint is named "lidar_joint", not "${frame}_joint".
-       sim_path forwarded like every other component's gz_frame_id. -->
+  <!-- Jackal's own bespoke gpu_lidar (link geometry, joint, gz sensor). joint_name
+       is separate from frame because jackal's joint is named "lidar_joint", not
+       "${frame}_joint". sim_path forwarded like every other component's gz_frame_id. -->
   <xacro:arg name="sim_path" default=""/>
   <xacro:macro name="jackal_lidar_mount" params="parent_link *origin frame:=lidar_link joint_name:=lidar_joint">
@@ -36,5 +34,5 @@
       <sensor name="gpu_lidar" type="gpu_lidar">
         <gz_frame_id>$(arg sim_path)/${frame}</gz_frame_id>
-        <pose>0 0 0.142 0 0 0</pose>
+        <pose>0 0 0 0 0 0</pose>
         <update_rate>10</update_rate>
         <lidar>

File: arena_robots/tests/golden/jackal_default.urdf (robot description, URDF)
Before this commit: robot jackal, 14 links, 13 joints
Joints:
- joint lidar_joint: origin xyz=0.0 0.0 0.14200000000000002 rpy=0 0 0 -> xyz=0.0 0.0 0.284 rpy=0 0 0

Commit message: fix fix jackal

File: arena_robots/components/lidar/jackal_default/lidar.urdf.xacro (robot description, xacro)
@@ -6,12 +6,13 @@
   <xacro:arg name="sim_path" default=""/>
   <xacro:macro name="jackal_lidar_mount" params="parent_link *origin frame:=lidar_link joint_name:=lidar_joint">
+    <xacro:property name="body_z" value="-0.142"/>
     <link name="${frame}">
       <inertial>
-        <origin xyz="0 0 0" rpy="0 0 0"/>
+        <origin xyz="0 0 ${body_z}" rpy="0 0 0"/>
         <mass value="0.1"/>
         <inertia ixx="1e-5" ixy="0" ixz="0" iyy="1e-5" iyz="0" izz="1e-5"/>
       </inertial>
       <visual>
-        <origin xyz="0 0 0" rpy="0 0 0"/>
+        <origin xyz="0 0 ${body_z}" rpy="0 0 0"/>
         <geometry>
           <cylinder radius="0.05" length="0.1"/>
@@ -20,5 +21,5 @@
       </visual>
       <collision>
-        <origin xyz="0 0 0" rpy="0 0 0"/>
+        <origin xyz="0 0 ${body_z}" rpy="0 0 0"/>
         <geometry>
           <cylinder radius="0.05" length="0.1"/>
